File: ramptronix/Uni-2.x/Uni-2.2,Complete.brd (EAGLE design)
At the start: 172 x 73.5 mm, 117 parts, among them IC1 UCC38083DR, IC2 MCP14A0304T-E_SN, IC4 ME3116, IC6 TL431CL3T, IC7 ME3116, J1 61300211121, J2 TB005-762-02BE, J3 TB005-762-02BE, Q1 STB130N6F7, Q2 STB130N6F7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

Commit message: Uni-2.2 HW Design Update EAGLE
Update
- Hole patterns
- LV Creapage/clearances
- PWR Plane stitching via locations
- PWR Plane routing
Parts:
- removed J2: TB005-762-02BE, SamacSys_Parts:TB00576202BE
- added INPUT: TB005-762-02BE, SamacSys_Parts:TB00576202BE
- moved U$1 10.8 mm to (164.9, 53.9)
- moved U$2 8.90 mm to (155.1, 20.8)
- moved HVLED 7.43 mm to (164.0, 15.0), turned to 180 degrees
- moved R33 7.21 mm to (46.5, 65.0)
- moved C36 6.40 mm to (52.1, 65.0)
- moved R26 6.25 mm to (8.18, 3.10), turned to 270 degrees
- moved PWRGND_TP 6.00 mm to (135.5, 7.00)
- moved U$3 5.70 mm to (157.4, 7.50)
- moved D6 5.62 mm to (74.5, 17.0), turned to 180 degrees
- moved R10 5.00 mm to (118.5, 12.0)
- moved R14 5.00 mm to (112.5, 12.0)
- moved R19 5.00 mm to (149.5, 12.0)
- moved R22 5.00 mm to (144.0, 12.0)
- moved R34 5.00 mm to (138.5, 12.0)
- moved R35 5.00 mm to (133.0, 12.0)
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Connections:
- net GNDA: now also INPUT.2; no longer J2.2
- net VCC28V: now also INPUT.1; no longer J2.1
Routing:
- net PWRGND: track 45.0 -> 133.0 mm, vias 122 -> 51
- net REG: track 28.2 -> 103.5 mm
- net VCC28V: track 11.0 -> 51.8 mm, vias 86 -> 101
- net AUX1: track 57.6 -> 82.0 mm
- net GNDA: track 39.4 -> 62.6 mm, vias 153 -> 131
- net TRANS2: track 5.94 -> 23.7 mm, vias 74 -> 70
- net TRANS1: track 13.5 -> 20.5 mm, vias 74 -> 70
- net OPTO-EMITT: track 16.0 -> 22.9 mm
- net Q2G: track 16.9 -> 23.5 mm, vias 6 -> 3
- net N$25: track 4.02 -> 8.99 mm
- net REG5V: track 51.0 -> 55.8 mm
- net SWITCH1: track 0.00 -> 3.48 mm
- net N$12: track 6.03 -> 9.26 mm
- net N$7: track 24.4 -> 27.0 mm
- net DRAIN2: track 41.8 -> 43.9 mm
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- removed copper zone on layer 16, net REG
Other:
- outline, holes or cut-outs redrawn
- board text added: "*** WARNING HV PRESENT ***"
- board text added: "+VBATT"
- board text added: "GND_HV"
- board text removed: "IF LIT HV PRESENT!"
- board text removed: "V+ IN"
