File: ramptronix/Uni-2.x/Uni-2,0,Complete.brd (EAGLE design)
At the start: 172 x 73.5 mm, 117 parts, among them IC1 UCC38083DR, IC2 MCP14A0304T-E_SN, IC4 ME3116, IC6 TL431CL3T, IC7 ME3116, J1 61300211121, J2 TB005-762-02BE, J3 TB005-762-02BE, Q1 STB130N6F7, Q2 STB130N6F7, T1 BIGTRANS, T1.2 B66362B1014T001

Commit message: Added Latest Board Revisions and Changelog.txt file
see title
Parts:
- removed GND_TP1: TPSQPAD1-13, testpad:P1-13
- removed HVLED: RED, led:CHIPLED_0805
- removed OPT1: VOL617A-4X001T, SamacSys_Parts:SOP254P1015X230-4N
- removed VR1: LM317MBDT, v-reg:DPACK
- added C19: ECW-FE2W105K, SamacSys_Parts:ECWFE2W105K
- added F1: 1206SMTFUSE, SamacSys_Parts:1206SMTFUSE
- added IC3: LM317MBDT, v-reg:DPACK
- added LED1: RED, led:CHIPLED_0805
- added Q5: VOL617A-4X001T, SamacSys_Parts:SOP254P1015X230-4N
- C15, C16: value 400BXW100MEFR18X25 -> EEU-ED2V470S; device SamacSys_Parts:CAPPRD750W80D1825H2700 -> SamacSys_Parts:CAPPRD750W85D1800H2200
- C17, C18: value C1812C274KCRACAUTO -> EEU-ED2V470S; device SamacSys_Parts:C1812 -> SamacSys_Parts:CAPPRD750W85D1800H2200
- moved C35 51.9 mm to (43.0, 61.0)
- moved R36 47.0 mm to (112.0, -1.50), turned to 0 degrees
- moved C17 37.0 mm to (166.0, 19.5), turned to 270 degrees
- moved R19 35.3 mm to (118.5, -1.50), turned to 0 degrees
- moved C23 32.4 mm to (13.9, 52.8), turned to 270 degrees
- moved U$3 29.7 mm to (124.4, 6.00)
- moved C16 29.4 mm to (166.0, 51.5), turned to 90 degrees
- moved U$1 26.3 mm to (145.0, 41.2)
- moved R22 24.0 mm to (125.0, -1.50), turned to 0 degrees
- moved C15 22.0 mm to (146.5, 19.5), turned to 270 degrees
- moved U$2 20.8 mm to (145.0, 29.5)
- moved C1 18.3 mm to (53.5, 6.50), turned to 0 degrees
- moved C18 17.4 mm to (146.5, 51.5)
- moved C3 16.9 mm to (6.50, 53.5)
- moved C4 16.8 mm to (6.50, 18.0)
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- renumbered 5VLED to REG5V, VR2 to PS1
Connections:
- removed net VCC28V: C23.2, C24.1, C3.1, C35.1, C4.1, C5.1, C6.1, IC7.5, J2.1, R26.1, T1.2.7, T1.4, T1.5
- new net 28VFUSE: C23.2, C24.1, C3.1, C35.1, C4.1, C5.1, C6.1, F1.2, IC7.5, R26.1, T1.2.7, T1.4, T1.5
- new net N$20: F1.1, J2.1
- net DC+: now also C19.2
- net GNDA: now also Q5.3; no longer GND_TP1.TP, OPT1.3
- net N$10: now also IC3.1; no longer VR1.1
- net N$12: now also LED1.A; no longer HVLED.A
- net N$18: now also Q5.2; no longer OPT1.2
- net N$19: now also Q5.1; no longer OPT1.1
- net OPTO-EMITT: now also Q5.4; no longer OPT1.4
- net PRE: now also IC3.3; no longer VR1.3
- net PWRGND: now also C19.1, LED1.C; no longer HVLED.C
- net REG: now also IC3.4; no longer VR1.4
Routing:
- net REG: track 28.2 -> 58.0 mm, vias 7 -> 6
- net DC+: track 21.9 -> 41.2 mm
- net VCC28V: track 8.78 -> 0.00 mm, vias 86 -> 0
- net GNDA: track 37.3 -> 44.6 mm, vias 153 -> 154
- net N$10: track 3.44 -> 10.3 mm
- net PRE: track 24.2 -> 18.2 mm
- net N$6: track 7.17 -> 10.8 mm
- net REG5V: track 51.0 -> 54.3 mm
- net 28VFUSE: track 0.00 -> 3.05 mm, vias 0 -> 97
- net PWRGND: track 45.0 -> 47.4 mm, vias 122 -> 123
- net N$5: track 42.1 -> 40.2 mm
- net OPTO-EMITT: track 16.0 -> 17.7 mm
- net N$18: track 26.1 -> 27.8 mm
- net N$17: track 2.66 -> 4.23 mm
- net N$15: track 3.16 -> 2.16 mm
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- added copper zone on layer 1, net 28VFUSE
- added copper zone on layer 16, net 28VFUSE
- added copper zone on layer 1, net N$1
- added copper zone on layer 1, net N$15
- added copper zone on layer 1, net N$20
- removed copper zone on layer 1, net N$7
- removed copper zone on layer 1, net VCC28V
- removed copper zone on layer 16, net VCC28V
Other:
- board size 172 x 73.5 mm -> 178.5 x 73.5 mm
- board text removed: "IF LIT HV PRESENT!"
