File: ramptronix/Uni-2.x/Uni-2,0,Complete.sch (EAGLE design)
At the start: 113 parts, among them IC1 MCP14A0304T-E_SN, IC2 UCC38083DR, IC3 ME3116, IC4 ME3116, IC5 TL431CL3T, J1 TB005-762-02BE, J2 61300211121, Q1 STB130N6F7, Q2 STB130N6F7, T1 BIGTRANS, T1.1 B66362B1014T001

Commit message: Added Latest Board Revisions and Changelog.txt file
see title
Parts:
- removed GND_TP1: TPSQPAD1-13, testpad:TPSQPAD1-13
- removed INPUT: TB005-762-02BE, SamacSys_Parts:TB005-762-02BE
- removed U$4: HV, RMP - HALF BRIDGE 0.0.1:HV
- removed VR1: LM317MBDT, v-reg:LM317MBDT
- removed VR2: AP2120N-5.0TRG1, SamacSys_Parts:AP2120N-5.0TRG1
- added C3: OVK151M1VTR-10131, SamacSys_Parts:OVK151M1VTR-10131
- added C36: (no value), rcl:C-EUC1210K
- added F1: 1206SMTFUSE, SamacSys_Parts:1206SMTFUSE
- added IC7: ME3116, SamacSys_Parts:ME3116
- added J3: TB005-762-02BE, SamacSys_Parts:TB005-762-02BE
- added PS2: NXE2S1205MC-R13, SamacSys_Parts:NXE2S1205MC-R13
- added R1: 1k, rcl:R-US_R0603
- added U$1, U$2: HV, RMP - HALF BRIDGE 0.0.1:HV
- C1, C13: value OVK151M1VTR-10131 -> 10 uF; device SamacSys_Parts:OVK151M1VTR-10131 -> rcl:C-EUC0603K; LCSC_PART (none) -> C440198
- C10: device rcl:C-EUC0805K -> rcl:C-EUC0603K
- C11: device rcl:C-EUC0805K -> rcl:C-EUC0603K; LCSC_PART C440198 -> (none)
- C12: value OVK151M1VTR-10131 -> 100 pF; device SamacSys_Parts:OVK151M1VTR-10131 -> rcl:C-EUC0402K; LCSC_PART (none) -> C1546
- C14: value 10 uF -> 470 pF; LCSC_PART C440198 -> C1620
- C15: value 0.1 uF -> EEU-ED2V470S; device rcl:C-EUC0603K -> SamacSys_Parts:EEU-ED2V470S; LCSC_PART C440198 -> (none)
- C16: value 470 pF -> EEU-ED2V470S; device rcl:C-EUC0603K -> SamacSys_Parts:EEU-ED2V470S; LCSC_PART C1620 -> (none)
- C17: value 2.2nF -> EEU-ED2V470S; device rcl:C-EUC0603K -> SamacSys_Parts:EEU-ED2V470S
- C18: value 470pF -> EEU-ED2V470S; device rcl:C-EUC0603K -> SamacSys_Parts:EEU-ED2V470S
- C19: value 100 pF -> ECW-FE2W105K; device rcl:C-EUC0402K -> SamacSys_Parts:ECW-FE2W105K; LCSC_PART C1546 -> (none)
- C2: value OVK151M1VTR-10131 -> 0.1 uF; device SamacSys_Parts:OVK151M1VTR-10131 -> rcl:C-EUC0603K; LCSC_PART (none) -> C440198
- C20: value 0.1 uF -> 470pF; LCSC_PART C14663 -> (none)
- C21: value 10 uF -> 2.2nF; device rcl:C-EUC0805K -> rcl:C-EUC0603K
- C22: device rcl:C-EUC0402 -> rcl:C-EUC0805K
- C23, C32: device rcl:C-EUC0603K -> rcl:C-EUC0805K
- C24: value 10 uF -> 1 uF
- C25: value 100 pF -> 10 uF; device rcl:C-EUC0402K -> rcl:C-EUC0603K; LCSC_PART C1546 -> C440198
- C26: value 1 uF -> 10 uF; device rcl:C-EUC0603K -> rcl:C-EUC0805K
- C30: value 10 uF -> 100 pF; device rcl:C-EUC0805K -> rcl:C-EUC0402K; LCSC_PART C440198 -> C1546
- C31: device rcl:C-EUC0805K -> rcl:C-EUC0402
- C33: LCSC_PART (none) -> C440198
- C34: device rcl:C-EUC0805K -> rcl:C-EUC0603K; LCSC_PART (none) -> C440198
- C35: value 10 uF -> 1 uF; device rcl:C-EUC0603K -> rcl:C-EUC0805K
- C4, C5: value C1812C274KCRACAUTO -> OVK151M1VTR-10131; device SamacSys_Parts:C1812C274KCRACAUTO -> SamacSys_Parts:OVK151M1VTR-10131
- C6: value 400BXW100MEFR18X25 -> OVK151M1VTR-10131; device SamacSys_Parts:400BXW100MEFR18X25 -> SamacSys_Parts:OVK151M1VTR-10131
- C7: value 400BXW100MEFR18X25 -> 10 uF; device SamacSys_Parts:400BXW100MEFR18X25 -> rcl:C-EUC0805K
- C8: value 1 uF -> 0.1 uF; device rcl:C-EUC0805K -> rcl:C-EUC0603K; LCSC_PART C440198 -> C14663
- C9: device rcl:C-EUC0603K -> rcl:C-EUC0805K; LCSC_PART C440198 -> (none)
- GATE1_TP, GATE2_TP: value TPTP13R -> TPSQPAD1-17; device testpad:TPTP13R -> testpad:TPSQPAD1-17
- IC1: value MCP14A0304T-E_SN -> UCC38083DR; device SamacSys_Parts:MCP14A0304T-E_SN -> SamacSys_Parts:UCC38083DR
- IC2: value UCC38083DR -> MCP14A0304T-E_SN; device SamacSys_Parts:UCC38083DR -> SamacSys_Parts:MCP14A0304T-E_SN
- IC3: value ME3116 -> LM317MBDT; device SamacSys_Parts:ME3116 -> v-reg:LM317MBDT; LCSC_PART C97643 -> (none)
- J1: value TB005-762-02BE -> 61300211121; device SamacSys_Parts:TB005-762-02BE -> Headers:61300211121
- J2: value 61300211121 -> TB005-762-02BE; device Headers:61300211121 -> SamacSys_Parts:TB005-762-02BE
- L1: value 2300LL-102-V-RC -> LQH5BPN6R8NT0L; device SamacSys_Parts:2300LL-102-V-RC -> SamacSys_Parts:LQH5BPN6R8NT0L
- L3: value LQH5BPN6R8NT0L -> 2300LL-102-V-RC; device SamacSys_Parts:LQH5BPN6R8NT0L -> SamacSys_Parts:2300LL-102-V-RC
- PS1: value NXE2S1205MC-R13 -> AP2120N-5.0TRG1; device SamacSys_Parts:NXE2S1205MC-R13 -> SamacSys_Parts:AP2120N-5.0TRG1
- R10: value 470 -> 100k; device rcl:R-US_R0603 -> rcl:R-US_R1206; LCSC_PART C22975 -> (none)
- R12: value 1k -> 22k; LCSC_PART C22975 -> C31850
- R13: value 22k -> 470k; LCSC_PART C31850 -> C25811
- R14: value 470k -> 100k; device rcl:R-US_R0603 -> rcl:R-US_R1206; LCSC_PART C25811 -> (none)
- R16: value 100 -> 2.2k; device rcl:R-US_R1206 -> rcl:R-US_R0805
- R17: value 100 -> 820; device rcl:R-US_R1206 -> rcl:R-US_R0603
- R18: value 10k -> 330; device rcl:R-US_R0402 -> rcl:R-US_R0805; LCSC_PART C25779 -> (none)
- R19: value 10k -> 20k; device rcl:R-US_R0402 -> rcl:R-US_R1206; LCSC_PART C25779 -> (none)
- R2: value 10 -> 1k; device rcl:R-US_R0805 -> rcl:R-US_R0402
- R20: value 100k -> 470; device rcl:R-US_R0402 -> rcl:R-US_R0603; LCSC_PART C25741 -> C22975; SPICEPREFIX R -> (none)
- R21: value 330 -> 4.7k; device rcl:R-US_R0805 -> rcl:R-US_R0603; LCSC_PART (none) -> C22975
- R22: value 2.2k -> 20k; device rcl:R-US_R0805 -> rcl:R-US_R1206
- R23: value 100k -> 100
- R24: value 100k -> 2k; device rcl:R-US_R1206 -> rcl:R-US_R0603; LCSC_PART (none) -> C22975
- R25: value 100k -> 10k; device rcl:R-US_R1206 -> rcl:R-US_R0402; LCSC_PART (none) -> C25779
- R26, R28: value 20k -> 100k; device rcl:R-US_R1206 -> rcl:R-US_R0402; LCSC_PART (none) -> C25741; SPICEPREFIX (none) -> R
- R27: value 20k -> 560; device rcl:R-US_R1206 -> rcl:R-US_R0402; LCSC_PART (none) -> C4177; SPICEPREFIX (none) -> R
- R29, R30: value 20k -> 10k; device rcl:R-US_R1206 -> rcl:R-US_R0402; LCSC_PART (none) -> C25779
- R31: value 560 -> 100; device rcl:R-US_R0402 -> rcl:R-US_R1206; LCSC_PART C4177 -> (none); SPICEPREFIX R -> (none)
- R32: value 10k -> 1k; device rcl:R-US_R0402 -> rcl:R-US_R0603; LCSC_PART C25779 -> C22975
- R33: value 100k -> (none); device rcl:R-US_R0402 -> rcl:R-US_R1206; LCSC_PART C25741 -> (none); SPICEPREFIX R -> (none)
- R34: value 2k -> 20k; device rcl:R-US_R0603 -> rcl:R-US_R1206; LCSC_PART C22975 -> (none)
- R35: value 820 -> 20k; device rcl:R-US_R0603 -> rcl:R-US_R1206
- R36: value 1k -> 20k; device rcl:R-US_R0603 -> rcl:R-US_R1206; LCSC_PART C22975 -> (none)
- R4: value 1k -> 10; device rcl:R-US_R0402 -> rcl:R-US_R0805
- R5, R6: value 0.05 -> 10; device rcl:R-US_R2512 -> rcl:R-US_R0805
- R7, R8: value 10 -> 0.05; device rcl:R-US_R0805 -> rcl:R-US_R2512
- R9: value 4.7k -> 100k; device rcl:R-US_R0603 -> rcl:R-US_R1206; LCSC_PART C22975 -> (none)
- renumbered 5VLED to REG5V, HVLED to LED1, IC5 to IC6, OPT1 to Q5, SJ100 to SJ1, T1.1 to T1.2
Connections:
- removed net VCC28V: C1.+, C11.2, C12.+, C13.+, C2.+, C26.1, C8.1, IC4.IN, INPUT.1, R33.1, T1.2.7, T1.4, T1.5
- new net 28VFUSE: C23.2, C24.1, C3.+, C35.1, C4.+, C5.+, C6.+, F1.2, IC7.IN, R26.1, T1.2.7, T1.4, T1.5
- new net N$20: F1.1, J2.1
- new net N$29: C36.1, R33.2
- net AUXB: now also C10.2, C12.1, C25.2, C31.2, PS1.VIN, R29.1; no longer C19.1, C22.2, C23.2, C24.2, R18.1, VR2.VIN
- net AUXD: now also C7.1, C9.1, IC4.IN, R23.2, R28.1, R31.2; no longer C21.1, C34.1, IC3.IN, R16.2, R17.2, R20.1
- net BRIDGEGND: now also R7.2, R8.2; no longer R5.2, R6.2
- net BS1: now also IC7.BS; no longer IC4.BS
- net BS2: now also C8.1, IC4.BS; no longer C20.1, IC3.BS
- net CS-IN: now also C14.1, IC1.CS; no longer C16.1, IC2.CS
- net DC+: now also C15.+, C16.+, C17.+, C18.+, C19.2, J3.2, L3.2, R35.2, R9.1; no longer C4.1, C5.1, C6.+, C7.+, J1.2, L1.2, R25.1, R26.2
- net DRAIN1: now also R33.1; no longer T1.2.5, T1.6
- net DRAIN2: now also C36.2; no longer T1.2.9, T1.3
- net EN1: now also IC7.EN, R26.2; no longer IC4.EN, R33.2
- net EN2: now also IC4.EN, R28.2; no longer IC3.EN, R20.2
- net FB1: now also C30.2, IC7.FB, R25.1, R27.1; no longer C25.2, IC4.FB, R31.1, R32.1
- net FB2: now also C12.2, IC4.FB, R29.2, R30.1; no longer C19.2, IC3.FB, R18.2, R19.1
- net GNDA: now also C1.2, C13.2, C2.2, C22.1, C23.1, C24.2, C26.1, C3.-, C33.1, C35.2, C4.-, C5.-, C6.-, IC7.GND, J2.2, PS2.-VIN, R12.2, R21.1, R24.1, R27.2, R7.1, R8.1; no longer C1.-, C10.1, C11.1, C12.-, C13.-, C15.2, C16.2, C2.-, C26.2, C30.1, C31.1, C8.2, C9.2, GND_TP1.TP, IC4.GND, INPUT.2, PS1.-VIN, R14.2, R31.2, R34.1, R5.1, R6.1, R9.1
- net N$1: now also R10.1, R9.2; no longer R24.1, R25.2
- net N$10: now also IC3.ADJ, R20.1, R21.2; no longer R10.1, R9.2, VR1.ADJ
- net N$11: now also C33.2, PS2._+VIN; no longer C32.2, PS1._+VIN
- net N$12: now also R36.1; no longer R30.1
- net N$13: now also IC1.ISET, R12.1; no longer IC2.ISET, R13.1
- net N$14: now also R19.1, R36.2; no longer R29.1, R30.2
- net N$15: now also R10.2, R14.1; no longer R23.1, R24.2
- net N$16: now also R16.1, R18.2; no longer R21.2, R22.1
- net N$17: now also R19.2, R22.1; no longer R28.1, R29.2
- net N$18: now also C20.2; no longer C18.2
- net N$19: now also R17.2; no longer R35.2
- net N$2: now also IC1.OUTA, IC2.INA; no longer IC1.INA, IC2.OUTA
- net N$21: now also C21.2; no longer C17.2
- net N$22: now also R24.2; no longer R34.2
- net N$24: now also R22.2, R34.1; no longer R27.1, R28.2
- net N$26: now also R32.2; no longer R36.2
- net N$27: now also R23.1, R31.1; no longer R16.1, R17.1
- net N$28: now also R34.2, R35.1; no longer R26.1, R27.2
- net N$3: now also C20.1, C21.1, J1.1, R14.2, R16.2; no longer C17.1, C18.1, J2.1, R22.2, R23.2
- net N$5: now also IC1.OUTB, IC2.INB; no longer IC1.INB, IC2.OUTB
- net N$6: now also IC2.ENA, IC2.ENB, R2.1; no longer IC1.ENA, IC1.ENB, R4.1
- net N$7: now also IC2.OUT1, R4.1; no longer IC1.OUT1, R2.1
- net N$8: now also IC2.OUT2, R5.1, R6.1; no longer IC1.OUT2, R7.1, R8.1
- net OPTO-EMITT: now also IC1.CTRL, R1.2; no longer IC2.CTRL, R12.2
- net PRE: now also C26.2, C30.1, IC3.IN, L1.2, R25.2; no longer C25.1, C30.2, L3.2, R32.2, VR1.IN
- net PWRGND: now also C10.1, C11.1, C15.-, C16.-, C17.-, C18.-, C19.1, C25.1, C31.1, C34.1, C7.2, C9.2, D4.A1, D4.A2, IC4.GND, J1.2, J3.1, PS1.GND, PS2.-VOUT, R18.1, R30.2, R32.1; no longer C21.2, C22.1, C23.1, C24.1, C33.1, C34.2, C35.1, C4.2, C5.2, C6.-, C7.-, D3.A1, D3.A2, IC3.GND, J1.1, J2.2, PS1.-VOUT, R19.2, R21.1, R36.1, VR2.GND
- net Q1G: now also R4.2; no longer R2.2
- net Q2G: now also R5.2, R6.2; no longer R7.2, R8.2
- net RECT: now also D3.K, L3.1; no longer D4.K, L1.1
- net REG: now also C1.1, C13.1, C2.1, C22.2, C32.2, IC3.OUT, R1.1, R2.2, R20.2; no longer C10.2, C14.1, C15.1, C31.2, C9.1, R10.2, R12.1, R4.2, VR1.OUT
- net REG5V: now also C11.2, C34.2, PS1.VOUT, PS2.+VOUT, R17.1; no longer C33.2, C35.2, PS1.+VOUT, R35.1, VR2.VOUT
- net RT: now also IC1.RT, R13.1; no longer IC2.RT, R14.1
- net SWITCH1: now also IC7.SW, L1.1; no longer IC4.SW, L3.1
- net SWITCH2: now also C8.2, IC4.SW; no longer C20.2, IC3.SW
- net TRANS1: now also D3.A1, D3.A2, D4.K; no longer D1.K, D2.A1, D2.A2
- net TRANS2: now also D1.K, D2.A1, D2.A2; no longer D3.K, D4.A1, D4.A2
Other:
- note added: "30A RATED SMT"
- note added: "47 uF Per"
- note added: "snubb"
- note removed: "0.27 uF ea (SOFT FLEX TERM)"
- note removed: "100 uF Per"
- note removed: "BYV29B-500,118 MURB2060CT"
- note removed: "DIODES SELECTION"
- note removed: "FET Selection:"
- note removed: "Power Input"
- note removed: "YJB200G06B STB130N6F7"
