File: ramptronix/Uni-2.x/Uni-2.1,Complete.brd (EAGLE design)
At the start: 178.5 x 73.5 mm, 118 parts, among them IC1 UCC38083DR, IC2 MCP14A0304T-E_SN, IC3 LM317MBDT, IC4 ME3116, IC6 TL431CL3T, IC7 ME3116, J1 61300211121, J2 TB005-762-02BE, J3 TB005-762-02BE, Q1 STB130N6F7, Q2 STB130N6F7, Q5 VOL617A-4X001T, T1 BIGTRANS, T1.2 B66362B1014T001

Commit message: Added Latest Board Revisions and Changelog.txt file
see title
Parts:
- removed C19: ECW-FE2W105K, SamacSys_Parts:ECWFE2W105K
- removed F1: 1206SMTFUSE, SamacSys_Parts:1206SMTFUSE
- removed IC3: LM317MBDT, v-reg:DPACK
- removed LED1: RED, led:CHIPLED_0805
- removed Q5: VOL617A-4X001T, SamacSys_Parts:SOP254P1015X230-4N
- added GND_TP1: TPSQPAD1-13, testpad:P1-13
- added HVLED: RED, led:CHIPLED_0805
- added OPT1: VOL617A-4X001T, SamacSys_Parts:SOP254P1015X230-4N
- added VR1: LM317MBDT, v-reg:DPACK
- C15, C16: value EEU-ED2V470S -> 400BXW100MEFR18X25; device SamacSys_Parts:CAPPRD750W85D1800H2200 -> SamacSys_Parts:CAPPRD750W80D1825H2700
- C17, C18: value EEU-ED2V470S -> C1812C274KCRACAUTO; device SamacSys_Parts:CAPPRD750W85D1800H2200 -> SamacSys_Parts:C1812
- moved C35 51.9 mm to (10.5, 20.5)
- moved R36 47.0 mm to (158.0, 8.00), turned to 180 degrees
- moved C17 37.0 mm to (158.1, 55.6), turned to 90 degrees
- moved R19 35.3 mm to (152.5, 8.00), turned to 180 degrees
- moved C23 32.4 mm to (21.5, 21.2), turned to 0 degrees
- moved U$3 29.7 mm to (153.9, 3.00)
- moved C16 29.4 mm to (146.5, 29.5), turned to 270 degrees
- moved U$1 26.3 mm to (159.5, 63.2)
- moved R22 24.0 mm to (147.0, 8.00), turned to 180 degrees
- moved C15 22.0 mm to (146.5, 41.5), turned to 90 degrees
- moved U$2 20.8 mm to (164.0, 21.0)
- moved C1 18.3 mm to (35.2, 4.88), turned to 90 degrees
- moved C18 17.4 mm to (163.4, 55.6)
- moved C3 16.9 mm to (22.5, 59.0)
- moved C4 16.8 mm to (22.5, 13.0)
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- renumbered PS1 to VR2, REG5V to 5VLED
Connections:
- removed net 28VFUSE: C23.2, C24.1, C3.1, C35.1, C4.1, C5.1, C6.1, F1.2, IC7.5, R26.1, T1.2.7, T1.4, T1.5
- removed net N$20: F1.1, J2.1
- new net VCC28V: C23.2, C24.1, C3.1, C35.1, C4.1, C5.1, C6.1, IC7.5, J2.1, R26.1, T1.2.7, T1.4, T1.5
- net DC+: no longer C19.2
- net GNDA: now also GND_TP1.TP, OPT1.3; no longer Q5.3
- net N$10: now also VR1.1; no longer IC3.1
- net N$12: now also HVLED.A; no longer LED1.A
- net N$18: now also OPT1.2; no longer Q5.2
- net N$19: now also OPT1.1; no longer Q5.1
- net OPTO-EMITT: now also OPT1.4; no longer Q5.4
- net PRE: now also VR1.3; no longer IC3.3
- net PWRGND: now also HVLED.C; no longer C19.1, LED1.C
- net REG: now also VR1.4; no longer IC3.4
Routing:
- net REG: track 58.0 -> 28.2 mm, vias 6 -> 7
- net DC+: track 41.2 -> 22.3 mm
- net VCC28V: track 0.00 -> 11.0 mm, vias 0 -> 86
- net N$10: track 10.3 -> 3.44 mm
- net PRE: track 18.2 -> 24.2 mm
- net GNDA: track 44.6 -> 39.4 mm, vias 154 -> 153
- net N$6: track 10.8 -> 7.17 mm
- net REG5V: track 54.3 -> 51.0 mm
- net 28VFUSE: track 3.05 -> 0.00 mm, vias 97 -> 0
- net PWRGND: track 47.4 -> 45.0 mm, vias 123 -> 122
- net N$5: track 40.2 -> 42.4 mm
- net OPTO-EMITT: track 17.7 -> 16.0 mm
- net N$18: track 27.8 -> 26.1 mm
- net N$17: track 4.23 -> 2.66 mm
- net N$15: track 2.16 -> 3.16 mm
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- added copper zone on layer 1, net N$7
- added copper zone on layer 1, net VCC28V
- added copper zone on layer 16, net VCC28V
- removed copper zone on layer 1, net 28VFUSE
- removed copper zone on layer 16, net 28VFUSE
- removed copper zone on layer 1, net N$1
- removed copper zone on layer 1, net N$15
- removed copper zone on layer 1, net N$20
Other:
- board size 178.5 x 73.5 mm -> 172 x 73.5 mm
- board text added: "IF LIT HV PRESENT!"
