File: ramptronix/Uni-2.x/Uni-2.1,Complete.sch (EAGLE design)
At the start: 116 parts, among them IC1 UCC38083DR, IC2 MCP14A0304T-E_SN, IC3 LM317MBDT, IC4 ME3116, IC6 TL431CL3T, IC7 ME3116, J1 61300211121, J2 TB005-762-02BE, J3 TB005-762-02BE, Q1 STB130N6F7, Q2 STB130N6F7, Q5 VOL617A-4X001T, T1 BIGTRANS, T1.2 B66362B1014T001

Commit message: Added Latest Board Revisions and Changelog.txt file
see title
Parts:
- removed C19: ECW-FE2W105K, SamacSys_Parts:ECW-FE2W105K
- removed F1: 1206SMTFUSE, SamacSys_Parts:1206SMTFUSE
- added GND_TP1: TPSQPAD1-13, testpad:TPSQPAD1-13
- C15, C16: value EEU-ED2V470S -> 400BXW100MEFR18X25; device SamacSys_Parts:EEU-ED2V470S -> SamacSys_Parts:400BXW100MEFR18X25
- C17, C18: value EEU-ED2V470S -> C1812C274KCRACAUTO; device SamacSys_Parts:EEU-ED2V470S -> SamacSys_Parts:C1812C274KCRACAUTO
- renumbered IC3 to VR1, LED1 to HVLED, PS1 to VR2, Q5 to OPT1, REG5V to 5VLED
Connections:
- removed net 28VFUSE: C23.2, C24.1, C3.+, C35.1, C4.+, C5.+, C6.+, F1.2, IC7.IN, R26.1, T1.2.7, T1.4, T1.5
- removed net N$20: F1.1, J2.1
- new net VCC28V: C23.2, C24.1, C3.+, C35.1, C4.+, C5.+, C6.+, IC7.IN, J2.1, R26.1, T1.2.7, T1.4, T1.5
- net DC+: now also C17.1, C18.1; no longer C17.+, C18.+, C19.2
- net GNDA: now also GND_TP1.TP
- net PWRGND: now also C17.2, C18.2; no longer C17.-, C18.-, C19.1
Other:
- note added: "0.27 uF ea (SOFT FLEX TERM)"
- note added: "100 uF Per"
- note added: "Power Input"
- note removed: "30A RATED SMT"
- note removed: "47 uF Per"
- moved on the sheet: C15, C16
