File: ramptronix/Uni-2.x/Uni-2.3.brd (EAGLE design)
At the start: 172 x 73.5 mm, 117 parts, among them IC1 MCP14A0304T-E_SN, IC2 UCC38083DR, IC3 ME3116, IC4 ME3116, IC5 TL431CL3T, J1 TB005-762-02BE, J2 61300211121, Q1 STB130N6F7, Q2 STB130N6F7, T1 BIGTRANS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

Commit message: Uni-2.3
Misc Changes.
Parts:
- removed C3: (no value), rcl:C1210K
- removed R1: (no value), rcl:R1206
- moved C8 38.0 mm to (15.8, 62.1)
- moved C11 17.4 mm to (19.5, 42.5), turned to 90 degrees
- moved PWRGND_TP 12.4 mm to (147.9, 7.55)
- moved HVOUT_TP 7.46 mm to (134.2, 7.55)
- moved C9 0.86 mm to (14.1, 24.8)
- moved R7 0.80 mm to (20.8, 27.7)
- moved R8 0.80 mm to (22.8, 27.7)
- moved C10 0.25 mm to (18.0, 25.0)
Connections:
- removed net N$29: C3.1, R1.2
- net DRAIN1: no longer R1.1
- net DRAIN2: no longer C3.2
Routing:
- net N$29: track 7.18 -> 0.00 mm
- net Q2G: track 27.1 -> 32.4 mm, vias 6 -> 8
- net DRAIN2: track 44.9 -> 40.4 mm, vias 103 -> 92
- net N$7: track 27.0 -> 23.0 mm, vias 6 -> 8
- net GNDA: track 65.9 -> 69.9 mm
- net VCC28V: track 51.6 -> 54.9 mm
- net REG: track 102.8 -> 99.8 mm, vias 7 -> 5
- net DC+: track 20.5 -> 23.2 mm

Commit message: Added Latest Board Revisions and Changelog.txt file
see title
Parts:
- added C3: 1uF, rcl:C1206K
- added C36: 1uf, rcl:C1206K
- added D10, D11: ES5GC, Diode:DIOM5226X290N
- added R37, R38: 510, rcl:R2512
- C10, C11, C14, C21, C22, C23, C24, C28, C29, C30, C31, C32, C33, C34, C35, C9: value 10 uF -> 10uF
- C15: value 0.1 uF -> 100nF
- C16: value 470 pF -> 470pF
- C20, C27: value 0.1 uF -> 1uF
- C26, C8: value 1 uF -> 1uF
- IC5: value TL431CL3T -> cl431
- VR1: value LM317MBDT -> LM317
Connections:
- new net N$20: C3.1, D10.1, R37.1
- new net N$23: C36.1, D11.1, R38.1
- net DRAIN1: now also D10.2
- net DRAIN2: now also D11.2
- net VCC28V: now also C3.2, C36.2, R37.2, R38.2
Routing:
- net VCC28V: track 54.9 -> 65.8 mm
- net N$20: track 0.00 -> 10.7 mm
- net N$23: track 0.00 -> 10.7 mm
