File: ramptronix/Uni-2.x/Uni-2.3.sch (EAGLE design)
At the start: 115 parts, among them IC1 MCP14A0304T-E_SN, IC2 UCC38083DR, IC3 ME3116, IC4 ME3116, IC5 TL431CL3T, J1 TB005-762-02BE, J2 61300211121, Q1 STB130N6F7, Q2 STB130N6F7, T1 BIGTRANS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

Commit message: Uni-2.3
Misc Changes.
Parts:
- removed C3: (no value), rcl:C-EUC1210K
- removed R1: (no value), rcl:R-US_R1206
Connections:
- removed net N$29: C3.1, R1.2
- net DRAIN1: no longer R1.1
- net DRAIN2: no longer C3.2
Other:
- note removed: "snubb"
- moved on the sheet: R5, R6
Changed lines of the file:
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@@
 <attribute name="LCSC_PART" value="C440198"/>
 </part>
-<part name="R1" library="rcl" library_urn="urn:adsk.eagle:library:334" deviceset="R-US_" device="R1206" package3d_urn="urn:adsk.eagle:package:23540/2">
-<spice>
-<pinmapping spiceprefix="R">
-<pinmap gate="G$1" pin="1" pinorder="1"/>
-<pinmap gate="G$1" pin="2" pinorder="2"/>
-</pinmapping>
-</spice>
-</part>
-<part name="C3" library="rcl" library_urn="urn:adsk.eagle:library:334" deviceset="C-EU" device="C1210K" package3d_urn="urn:adsk.eagle:package:23683/2"/>
 <part name="HVOUT_TP" library="testpad" library_urn="urn:adsk.eagle:library:385" deviceset="TPSQ" device="PAD1-13" package3d_urn="urn:adsk.eagle:package:27946/1"/>
 <part name="J2" library="Headers" deviceset="61300211121" device="" package3d_urn="urn:adsk.eagle:package:11390690/2"/>
@@
 <wire x1="124.46" y1="91.44" x2="124.46" y2="27.94" width="0.1524" layer="97" style="longdash"/>
 <wire x1="254" y1="91.44" x2="254" y2="27.94" width="0.1524" layer="97" style="longdash"/>
-<text x="55.88" y="38.1" size="1.778" layer="91">snubb</text>
 <text x="127" y="55.88" size="1.778" layer="91">injection</text>
 <polygon width="0.1524" layer="117">
@@
 <instance part="SUPPLY4" gate="GND" x="154.94" y="152.4" smashed="yes"/>
 <instance part="SUPPLY5" gate="GND" x="154.94" y="109.22" smashed="yes"/>
-<instance part="R1" gate="G$1" x="53.34" y="33.02" smashed="yes">
-<attribute name="NAME" x="49.53" y="34.5186" size="1.778" layer="95"/>
-<attribute name="VALUE" x="49.53" y="29.718" size="1.778" layer="96"/>
-</instance>
-<instance part="C3" gate="G$1" x="66.04" y="33.02" smashed="yes" rot="R90">
-<attribute name="NAME" x="65.659" y="34.544" size="1.778" layer="95" rot="R90"/>
-<attribute name="VALUE" x="70.739" y="34.544" size="1.778" layer="96" rot="R90"/>
-</instance>
 <instance part="HVOUT_TP" gate="G$1" x="228.6" y="149.86" smashed="yes" rot="R180">
 <attribute name="NAME" x="233.68" y="154.305" size="1.778" layer="95" rot="R180"/>
@@
 <junction x="50.8" y="60.96"/>
 </segment>
-<segment>
-<pinref part="C3" gate="G$1" pin="2"/>
-<wire x1="71.12" y1="33.02" x2="81.28" y2="33.02" width="0.1524" layer="91"/>
-<label x="73.66" y="33.02" size="1.778" layer="95"/>
-</segment>
 </net>
 <net name="DRAIN1" class="0">
@@
 <wire x1="50.8" y1="68.58" x2="50.8" y2="71.12" width="0.1524" layer="91"/>
 <junction x="50.8" y="71.12"/>
-</segment>
-<segment>
-<pinref part="R1" gate="G$1" pin="1"/>
-<wire x1="48.26" y1="33.02" x2="38.1" y2="33.02" width="0.1524" layer="91"/>
-<label x="35.56" y="33.02" size="1.778" layer="95"/>
 </segment>
 </net>
@@
 <wire x1="83.82" y1="66.04" x2="109.22" y2="66.04" width="0.1524" layer="91"/>
 <label x="99.06" y="66.04" size="1.778" layer="95"/>
-</segment>
-</net>
-<net name="N$29" class="0">
-<segment>
-<pinref part="R1" gate="G$1" pin="2"/>
-<pinref part="C3" gate="G$1" pin="1"/>
-<wire x1="58.42" y1="33.02" x2="63.5" y2="33.02" width="0.1524" layer="91"/>
 </segment>
 </net>
@@
 <attribute name="VALUE" x="186.69" y="69.85" size="1.778" layer="96" align="center-left"/>
 </instance>
-<instance part="GND6" gate="1" x="228.6" y="68.58" smashed="yes"/>
+<instance part="GND6" gate="1" x="246.38" y="66.04" smashed="yes"/>
 <instance part="R3" gate="G$1" x="162.56" y="104.14" smashed="yes">
 <attribute name="NAME" x="158.75" y="105.6386" size="1.778" layer="95"/>
@@
 <attribute name="LCSC_PART" x="86.36" y="149.86" size="1.778" layer="96" display="off"/>
 </instance>
-<instance part="R6" gate="G$1" x="223.52" y="93.98" smashed="yes" rot="R90">
-<attribute name="NAME" x="222.0214" y="90.17" size="1.778" layer="95" rot="R90"/>
-<attribute name="VALUE" x="226.822" y="90.17" size="1.778" layer="96" rot="R90"/>
-</instance>
-<instance part="R5" gate="G$1" x="233.68" y="93.98" smashed="yes" rot="R90">
-<attribute name="NAME" x="232.1814" y="90.17" size="1.778" layer="95" rot="R90"/>
-<attribute name="VALUE" x="236.982" y="90.17" size="1.778" layer="96" rot="R90"/>
+<instance part="R6" gate="G$1" x="241.3" y="91.44" smashed="yes" rot="R90">
+<attribute name="NAME" x="239.8014" y="87.63" size="1.778" layer="95" rot="R90"/>
+<attribute name="VALUE" x="244.602" y="87.63" size="1.778" layer="96" rot="R90"/>
+</instance>
+<instance part="R5" gate="G$1" x="251.46" y="91.44" smashed="yes" rot="R90">
+<attribute name="NAME" x="249.9614" y="87.63" size="1.778" layer="95" rot="R90"/>
+<attribute name="VALUE" x="254.762" y="87.63" size="1.778" layer="96" rot="R90"/>
 </instance>
 <instance part="GND7" gate="1" x="124.46" y="137.16" smashed="yes"/>
@@
 </segment>
 <segment>
-<wire x1="228.6" y1="83.82" x2="228.6" y2="71.12" width="0.1524" layer="91"/>
-<label x="228.6" y="73.66" size="1.778" layer="95" rot="R90"/>
+<wire x1="246.38" y1="81.28" x2="246.38" y2="68.58" width="0.1524" layer="91"/>
+<label x="246.38" y="71.12" size="1.778" layer="95" rot="R90"/>
 <pinref part="GND6" gate="1" pin="GNDA"/>
 <pinref part="R6" gate="G$1" pin="1"/>
-<wire x1="228.6" y1="83.82" x2="223.52" y2="83.82" width="0.1524" layer="91"/>
-<wire x1="223.52" y1="83.82" x2="223.52" y2="88.9" width="0.1524" layer="91"/>
+<wire x1="246.38" y1="81.28" x2="241.3" y2="81.28" width="0.1524" layer="91"/>
+<wire x1="241.3" y1="81.28" x2="241.3" y2="86.36" width="0.1524" layer="91"/>
 <pinref part="R5" gate="G$1" pin="1"/>
-<wire x1="233.68" y1="88.9" x2="233.68" y2="83.82" width="0.1524" layer="91"/>
-<wire x1="233.68" y1="83.82" x2="228.6" y2="83.82" width="0.1524" layer="91"/>
-<junction x="228.6" y="83.82"/>
+<wire x1="251.46" y1="86.36" x2="251.46" y2="81.28" width="0.1524" layer="91"/>
+<wire x1="251.46" y1="81.28" x2="246.38" y2="81.28" width="0.1524" layer="91"/>
+<junction x="246.38" y="81.28"/>
 </segment>
 <segment>
@@
 <net name="BRIDGEGND" class="0">
 <segment>
-<wire x1="228.6" y1="104.14" x2="228.6" y2="119.38" width="0.1524" layer="91"/>
-<wire x1="228.6" y1="119.38" x2="223.52" y2="119.38" width="0.1524" layer="91"/>
-<label x="223.52" y="119.38" size="1.778" layer="95"/>
+<wire x1="246.38" y1="101.6" x2="246.38" y2="116.84" width="0.1524" layer="91"/>
+<wire x1="246.38" y1="116.84" x2="241.3" y2="116.84" width="0.1524" layer="91"/>
+<label x="241.3" y="116.84" size="1.778" layer="95"/>
 <pinref part="R6" gate="G$1" pin="2"/>
-<wire x1="223.52" y1="99.06" x2="223.52" y2="104.14" width="0.1524" layer="91"/>
-<wire x1="223.52" y1="104.14" x2="228.6" y2="104.14" width="0.1524" layer="91"/>
+<wire x1="241.3" y1="96.52" x2="241.3" y2="101.6" width="0.1524" layer="91"/>
+<wire x1="241.3" y1="101.6" x2="246.38" y2="101.6" width="0.1524" layer="91"/>
 <pinref part="R5" gate="G$1" pin="2"/>
-<wire x1="233.68" y1="99.06" x2="233.68" y2="104.14" width="0.1524" layer="91"/>
-<wire x1="233.68" y1="104.14" x2="228.6" y2="104.14" width="0.1524" layer="91"/>
-<junction x="228.6" y="104.14"/>
-</segment>
-<segment>
+<wire x1="251.46" y1="96.52" x2="251.46" y2="101.6" width="0.1524" layer="91"/>
+<wire x1="251.46" y1="101.6" x2="246.38" y2="101.6" width="0.1524" layer="91"/>
+<junction x="246.38" y="101.6"/>
+</segment>
+<segment>

Commit message: Added Latest Board Revisions and Changelog.txt file
see title
Parts:
- added C3: 1uF, rcl:C-EUC1206K
- added C36: 1uf, rcl:C-EUC1206K
- added D10, D11: ES5GC, Diode:DIODEDO-214AC(SMA)
- added R37, R38: 510, rcl:R-US_R2512
- C10, C11, C14, C21, C22, C23, C24, C28, C29, C30, C31, C32, C33, C34, C35, C9: value 10 uF -> 10uF
- C15: value 0.1 uF -> 100nF
- C16: value 470 pF -> 470pF
- C20, C27: value 0.1 uF -> 1uF
- C26, C8: value 1 uF -> 1uF
- IC5: value TL431CL3T -> cl431
- VR1: value LM317MBDT -> LM317
Connections:
- new net N$20: C3.1, D10.C, R37.1
- new net N$23: C36.1, D11.C, R38.1
- net DRAIN1: now also D10.A
- net DRAIN2: now also D11.A
- net VCC28V: now also C3.2, C36.2, R37.2, R38.2
