File: ramptronix/Uni-2.x/Uni-2.31.brd (EAGLE design)
At the start: 172 x 73.5 mm, 117 parts, among them IC1 MCP14A0304T-E_SN, IC2 UCC38083DR, IC3 ME3116, IC4 ME3116, IC5 TL431CL3T, J1 TB005-762-02BE, J2 61300211121, Q1 STB130N6F7, Q2 STB130N6F7, T1 BIGTRANS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

Commit message: Added Latest Board Revisions and Changelog.txt file
see title
Parts:
- removed R1: (no value), rcl:R1206
- added C36: 1uF, rcl:C1206K
- added D10, D11: ES5G, Diode:DIOM5336X265N
- added R37, R38: 510, rcl:R2512
- C10: value 10 uF -> 100nF; device rcl:C0805K -> rcl:C0402
- C11, C14, C21, C23, C24, C33, C34, C35, C9: value 10 uF -> 10uF
- C15: value 0.1 uF -> 100nF; device rcl:C0603K -> rcl:C0402
- C16: value 470 pF -> 470pF
- C20, C27: value 0.1 uF -> 1uF
- C22, C32: value 10 uF -> 1uF
- C26, C8: value 1 uF -> 1uF
- C28, C30, C31: value 10 uF -> 10uF; device rcl:C0805K -> rcl:C0603K
- C29: value 10 uF -> 1uF; device rcl:C0805K -> rcl:C0603K
- C3: value (none) -> 1uF; device rcl:C1210K -> rcl:C1206K
- D1, D2, D3, D4: value FERD20H60CG-TR -> MURB1060CT
- GATE1_TP, GATE2_TP: value TPSQPAD1-17 -> TPTP13R; device testpad:P1-17 -> testpad:TP13R
- IC5: value TL431CL3T -> cl431
- R19: value 10k -> 2k
- R20, R33: value 100k -> 1M
- R31: device rcl:R0402 -> rcl:R0603
- VR1: value LM317MBDT -> LM317
- moved C8 43.9 mm to (15.8, 68.1)
- moved PWRGND_TP 12.4 mm to (147.9, 7.55)
- moved C3 8.63 mm to (45.9, 70.9), turned to 180 degrees
- moved HVOUT_TP 7.46 mm to (134.2, 7.55)
- moved C9 6.29 mm to (15.4, 31.5)
- moved R4 6.20 mm to (11.6, 36.8)
- moved T1.1 6.19 mm to (52.4, 61.1)
- moved C10 6.17 mm to (19.9, 31.1), turned to 0 degrees
- moved T1 6.02 mm to (47.5, 28.5)
- moved C1 6.00 mm to (22.5, 69.0)
- moved C12 6.00 mm to (22.5, 23.0)
- moved C13 6.00 mm to (35.0, 23.0)
- moved C2 6.00 mm to (35.0, 69.0)
- moved C4 6.00 mm to (158.1, 65.6)
- moved C5 6.00 mm to (163.4, 65.6)
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Connections:
- removed net N$29: C3.1, R1.2
- new net N$20: C3.1, D10.1, R37.1
- new net N$23: C36.1, D11.1, R38.1
- net DRAIN1: now also D10.2, T1.1.5, T1.6; no longer R1.1
- net DRAIN2: now also D11.2, T1.1.9, T1.3; no longer C3.2
- net GNDA: now also C10.2; no longer C10.1
- net REG: now also C10.1; no longer C10.2
- net VCC28V: now also C3.2, C36.2, R37.2, R38.2
Routing:
- net DRAIN2: track 43.9 -> 0.14 mm, vias 0 -> 113
- net AUX1: track 82.0 -> 57.6 mm
- net N$7: track 27.0 -> 5.50 mm, vias 6 -> 8
- net REG: track 103.5 -> 123.0 mm, vias 7 -> 5
- net VCC28V: track 51.8 -> 70.2 mm
- net PWRGND: track 133.0 -> 120.1 mm, vias 51 -> 52
- net Q2G: track 23.5 -> 32.4 mm, vias 3 -> 8
- net DC+: track 20.5 -> 29.2 mm
- net BRIDGEGND: track 27.8 -> 35.7 mm, vias 0 -> 2
- net N$23: track 0.00 -> 7.57 mm
- net N$2: track 49.5 -> 55.0 mm
- net GNDA: track 65.9 -> 71.4 mm, vias 130 -> 143
- net N$5: track 44.0 -> 49.3 mm
- net N$20: track 0.00 -> 4.12 mm
- net N$29: track 2.78 -> 0.00 mm
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- added copper zone on layer 16, net DRAIN1
- added copper zone on layer 16, net DRAIN2
- added copper zone on layer 1, net N$20
- added copper zone on layer 1, net N$23
Other:
- board size 172 x 73.5 mm -> 172 x 79.5 mm
- board text added: "ABS MAX 35V IN"
