File: ramptronix/Uni-2.x/Uni-2.31.sch (EAGLE design)
At the start: 115 parts, among them IC1 MCP14A0304T-E_SN, IC2 UCC38083DR, IC3 ME3116, IC4 ME3116, IC5 TL431CL3T, J1 TB005-762-02BE, J2 61300211121, Q1 STB130N6F7, Q2 STB130N6F7, T1 BIGTRANS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

Commit message: Added Latest Board Revisions and Changelog.txt file
see title
Parts:
- removed R1: (no value), rcl:R-US_R1206
- added C36: 1uF, rcl:C-EUC1206K
- added D10, D11: ES5G, Diode:DIODEDO-214AA(SMB)
- added R37, R38: 510, rcl:R-US_R2512
- C10: value 10 uF -> 100nF; device rcl:C-EUC0805K -> rcl:C-EUC0402
- C11, C14, C21, C23, C24, C33, C34, C35, C9: value 10 uF -> 10uF
- C15: value 0.1 uF -> 100nF; device rcl:C-EUC0603K -> rcl:C-EUC0402
- C16: value 470 pF -> 470pF
- C20, C27: value 0.1 uF -> 1uF
- C22, C32: value 10 uF -> 1uF
- C26, C8: value 1 uF -> 1uF
- C28, C30, C31: value 10 uF -> 10uF; device rcl:C-EUC0805K -> rcl:C-EUC0603K
- C29: value 10 uF -> 1uF; device rcl:C-EUC0805K -> rcl:C-EUC0603K
- C3: value (none) -> 1uF; device rcl:C-EUC1210K -> rcl:C-EUC1206K
- D1, D2, D3, D4: value FERD20H60CG-TR -> MURB1060CT
- GATE1_TP, GATE2_TP: value TPSQPAD1-17 -> TPTP13R; device testpad:TPSQPAD1-17 -> testpad:TPTP13R
- IC5: value TL431CL3T -> cl431
- R19: value 10k -> 2k
- R20, R33: value 100k -> 1M
- R31: device rcl:R-US_R0402 -> rcl:R-US_R0603
- VR1: value LM317MBDT -> LM317
Connections:
- removed net N$29: C3.1, R1.2
- new net N$20: C3.1, D10.C, R37.1
- new net N$23: C36.1, D11.C, R38.1
- net DRAIN1: now also D10.A, T1.1.5, T1.6; no longer R1.1
- net DRAIN2: now also D11.A, T1.1.9, T1.3; no longer C3.2
- net GNDA: now also C10.2; no longer C10.1
- net REG: now also C10.1; no longer C10.2
- net VCC28V: now also C3.2, C36.2, R37.2, R38.2
Other:
- note added: "DIODES SELECTION"
- note added: "FET Selection:"
- note added: "YJB200G06B STB130N6F7"
- note removed: "snubb"
- moved on the sheet: R5, R6
