File: ramptronix/Uni-2.x/Uni-2.32.brd (EAGLE design)
At the start: 172 x 73.5 mm, 115 parts, among them IC1 MCP14A0304T-E_SN, IC2 UCC38083DR, IC3 ME3116, IC4 ME3116, IC5 TL431CL3T, J1 TB005-762-02BE, J2 61300211121, Q1 STB130N6F7, Q2 STB130N6F7, T1 BIGTRANS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

Commit message: Added Latest Board Revisions and Changelog.txt file
see title
Parts:
- removed SJ100: (no value), jumper:SJ_2W
- added C3, C36: 1uF, rcl:C1206K
- added D10, D11: ES5G, Diode:DIOM5336X265N
- added R37, R38: 510, rcl:R2512
- C10: value 10 uF -> 100nF; device rcl:C0805K -> rcl:C0402
- C11, C14, C21, C23, C24, C33, C34, C35, C9: value 10 uF -> 10uF
- C15: value 0.1 uF -> 100nF; device rcl:C0603K -> rcl:C0402
- C16: value 470 pF -> 470pF
- C17: value 2.2nF -> 47nF
- C20, C27: value 0.1 uF -> 1uF
- C22, C32: value 10 uF -> 1uF
- C26, C8: value 1 uF -> 1uF
- C28, C30, C31: value 10 uF -> 10uF; device rcl:C0805K -> rcl:C0603K
- C29: value 10 uF -> 1uF; device rcl:C0805K -> rcl:C0603K
- D1, D2, D3, D4: value FERD20H60CG-TR -> SICDIODE; device SamacSys_Parts:STB20N95K5 -> SamacSys_Parts:TO-252
- IC5: value TL431CL3T -> cl431
- R14: value 470k -> 220k
- R15: value 15k -> 33k
- R19: value 10k -> 2k
- R20, R33: value 100k -> 1M
- R31: value 560 -> 470; device rcl:R0402 -> rcl:R0603
- R35: value 820 -> 620
- VR1: value LM317MBDT -> LM317
- moved D2 140.3 mm to (-14.0, -18.0)
- moved D4 139.4 mm to (-14.0, -36.0), turned to 0 degrees
- moved D1 123.0 mm to (-14.0, -9.00), turned to 0 degrees
- moved D3 122.6 mm to (-14.0, -27.0)
- moved C8 43.9 mm to (15.8, 68.1)
- moved PWRGND_TP 12.4 mm to (147.9, 7.55)
- moved HVOUT_TP 7.46 mm to (134.2, 7.55)
- moved C9 6.29 mm to (15.4, 31.5)
- moved T1.1 6.19 mm to (52.4, 61.1)
- moved C10 6.17 mm to (19.9, 31.1), turned to 0 degrees
- moved T1 6.02 mm to (47.5, 28.5)
- moved R4 6.00 mm to (11.6, 36.8)
- moved C1 6.00 mm to (22.5, 69.0)
- moved C12 6.00 mm to (22.5, 23.0)
- moved C13 6.00 mm to (35.0, 23.0)
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Connections:
- removed net N$25: SJ100.3, T1.13
- removed net N$9: SJ100.1, T1.11
- new net N$20: C3.1, D10.1, R37.1
- new net N$23: C36.1, D11.1, R38.1
- net DRAIN1: now also D10.2
- net DRAIN2: now also D11.2
- net GNDA: now also C10.2; no longer C10.1
- net PWRGND: now also D1.2, D3.2; no longer D1.1, D1.3, D3.1, D3.3
- net RECT: now also D2.1, D2.3, D4.1, D4.3; no longer D2.2, D4.2
- net REG: now also C10.1; no longer C10.2
- net TRANS1: now also D1.1, D1.3, D2.2, T1.11; no longer D1.2, D2.1, D2.3, SJ100.2
- net TRANS2: now also D3.1, D3.3, D4.2; no longer D3.2, D4.1, D4.3
- net VCC28V: now also C3.2, C36.2, R37.2, R38.2
Routing:
- net DRAIN2: track 40.4 -> 0.14 mm, vias 12 -> 113
- net N$7: track 27.0 -> 5.50 mm, vias 6 -> 8
- net REG: track 102.8 -> 123.0 mm, vias 7 -> 5
- net VCC28V: track 51.6 -> 70.2 mm
- net PWRGND: track 133.0 -> 114.9 mm, vias 51 -> 52
- net N$25: track 8.99 -> 0.00 mm
- net Q2G: track 23.5 -> 32.4 mm, vias 6 -> 8
- net DC+: track 20.5 -> 29.2 mm
- net BRIDGEGND: track 27.8 -> 35.7 mm, vias 0 -> 2
- net AUX1: track 49.9 -> 57.6 mm
- net N$23: track 0.00 -> 7.57 mm
- net N$9: track 7.50 -> 0.00 mm
- net N$2: track 49.5 -> 55.0 mm
- net GNDA: track 65.9 -> 71.4 mm, vias 130 -> 143
- net N$5: track 44.0 -> 49.3 mm
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- added copper zone on layer 1, net N$20
- added copper zone on layer 1, net N$23
Other:
- board size 172 x 73.5 mm -> 172 x 79.5 mm
- board text added: "ABS MAX 35V IN"
