File: ramptronix/Uni-2.x/Uni-2.4.sch (EAGLE design)
At the start: 115 parts, among them IC1 MCP14A0304T-E_SN, IC2 UCC38083DR, IC3 ME3116, IC4 ME3116, IC5 TL431CL3T, J1 TB005-762-02BE, J2 61300211121, Q1 STB130N6F7, Q2 STB130N6F7, T1 BIGTRANS, T1.1 B66362B1014T001

Commit message: Added Latest Board Revisions and Changelog.txt file
see title
Parts:
- removed C35: 10 uF, rcl:C-EUC0603K
- removed D8, D9: SM4007PL, SamacSys_Parts:1N4148W-7-F
- removed PS1: NXE2S1205MC-R13, SamacSys_Parts:NXE2S1205MC-R13
- removed R1: (no value), rcl:R-US_R1206
- removed SJ100: (no value), jumper:SJ2WW
- added C36: 1uF, rcl:C-EUC1206K
- added D10, D11: ES5G, Diode:DIODEDO-214AA(SMB)
- added L4: LQH5BPN6R8NT0L, SamacSys_Parts:LQH5BPN6R8NT0L
- added R37, R38: 510, rcl:R-US_R2512
- C10: value 10 uF -> 100nF; device rcl:C-EUC0805K -> rcl:C-EUC0402
- C11, C14, C21, C23, C24, C32, C33, C34, C9: value 10 uF -> 10uF
- C15: value 0.1 uF -> 100nF; device rcl:C-EUC0603K -> rcl:C-EUC0402
- C16: value 470 pF -> 470pF
- C17: value 2.2nF -> 47nF
- C20, C27: value 0.1 uF -> 1uF
- C22: value 10 uF -> 1uF
- C26, C8: value 1 uF -> 1uF
- C28, C30, C31: value 10 uF -> 10uF; device rcl:C-EUC0805K -> rcl:C-EUC0603K
- C29: value 10 uF -> 1uF; device rcl:C-EUC0805K -> rcl:C-EUC0603K
- C3: value (none) -> 1uF; device rcl:C-EUC1210K -> rcl:C-EUC1206K
- D1, D2, D3, D4: value FERD20H60CG-TR -> C967703; device SamacSys_Parts:FERD20H60CG-TR -> SamacSys_Parts:SICDIODE
- GATE1_TP, GATE2_TP: value TPSQPAD1-17 -> TPTP13R; device testpad:TPSQPAD1-17 -> testpad:TPTP13R
- IC3, IC4: value ME3116 -> BD9G101G-TR; device SamacSys_Parts:ME3116 -> SamacSys_Parts:BD9G101G-TR
- IC5: value TL431CL3T -> cl431
- R15: value 15k -> 33k
- R19: value 10k -> 2k
- R20, R33: value 100k -> 1M
- R31: value 560 -> 470; device rcl:R-US_R0402 -> rcl:R-US_R0603
- R35: value 820 -> 1k
- VR1: value LM317MBDT -> LM317
Connections:
- removed net N$11: C32.2, D9.K, PS1._+VIN
- removed net N$25: SJ100.3, T1.13
- removed net N$29: C3.1, R1.2
- removed net N$4: D8.K, D9.A
- removed net N$9: SJ100.1, T1.11
- removed net VCC28V: C1.+, C11.2, C12.+, C13.+, C2.+, C26.1, C8.1, IC4.IN, INPUT.1, R33.1, T1.1.7, T1.4, T1.5
- new net AUXBFILT: C24.2, C32.2, L4.P$2, VR2.VIN
- new net N$20: C3.1, D10.C, R37.1
- new net N$23: C36.1, D11.C, R38.1
- new net VCCIN: C1.+, C11.2, C12.+, C13.+, C2.+, C26.1, C3.2, C36.2, C8.1, IC4.IN, INPUT.1, R33.1, R37.2, R38.2, T1.1.7, T1.4, T1.5
- net AUXB: now also L3.P$2, L4.P$1; no longer C24.2, L2.1, VR2.VIN
- net DRAIN1: now also D10.A, T1.1.5; no longer R1.1
- net DRAIN2: now also D11.A, T1.1.9; no longer C3.2
- net GNDA: now also C10.2; no longer C10.1, C32.1, PS1.-VIN
- net PRE: now also L2.P$2; no longer L3.2
- net PWRGND: now also C32.1, D1.A, D4.A; no longer C35.1, D1.A1, D1.A2, D3.A1, D3.A2, PS1.-VOUT
- net RECT: now also D2.K_1, D2.K_2, D3.K_1, D3.K_2; no longer D2.K, D4.K
- net REG: now also C10.1; no longer C10.2, D8.A
- net REG5V: no longer C35.2, PS1.+VOUT
- net SWITCH1: now also L2.P$1; no longer L3.1
- net SWITCH2: now also L3.P$1; no longer L2.2
- net TRANS1: now also D1.K_1, D1.K_2, D2.A, T1.11; no longer D1.K, D2.A1, D2.A2, SJ100.2
- net TRANS2: now also D3.A, D4.K_1, D4.K_2; no longer D3.K, D4.A1, D4.A2
Other:
- note added: "Pay Attention to 431 Pinout!!!!!"
- note removed: "BYV29B-500,118 MURB2060CT"
- note removed: "snubb"
- moved on the sheet: 5VLED, C22, C23, C24, C32, D5, D6, D7, R10, R36, R5, R6
