File: ramptronix/Uni-4-Layers/Uni4lay-1.0.brd (EAGLE design)
At the start: 172 x 73.5 mm, 117 parts, among them IC1 MCP14A0304T-E_SN, IC2 UCC38083DR, IC3 ME3116, IC4 ME3116, IC5 TL431CL3T, J1 TB005-762-02BE, J2 61300211121, Q1 STB130N6F7, Q2 STB130N6F7, T1 BIGTRANS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

Commit message: Uni-2.3
Misc Changes.
Parts:
- removed C3: (no value), rcl:C1210K
- removed R1: (no value), rcl:R1206
Connections:
- removed net N$29: C3.1, R1.2
- net DRAIN1: no longer R1.1
- net DRAIN2: no longer C3.2
Routing:
- net N$29: track 7.18 -> 0.00 mm
- net DRAIN2: track 44.9 -> 40.4 mm, vias 103 -> 12
- net Q2G: track 27.1 -> 23.5 mm
- added copper zone on layer 15, net GNDA
- added copper zone on layer 2, net VCC28V
- removed copper zone on layer 16, net VCC28V
