File: ramptronix/Uni-4-Layers/Uni4lay-1.0.sch (EAGLE design)
At the start: 115 parts, among them IC1 MCP14A0304T-E_SN, IC2 UCC38083DR, IC3 ME3116, IC4 ME3116, IC5 TL431CL3T, J1 TB005-762-02BE, J2 61300211121, Q1 STB130N6F7, Q2 STB130N6F7, T1 BIGTRANS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

Commit message: Uni-2.3
Misc Changes.
Parts:
- removed C3: (no value), rcl:C-EUC1210K
- removed R1: (no value), rcl:R-US_R1206
Connections:
- removed net N$29: C3.1, R1.2
- net DRAIN1: no longer R1.1
- net DRAIN2: no longer C3.2
Other:
- note removed: "snubb"
- moved on the sheet: R5, R6
Changed lines of the file:
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@@
 <attribute name="LCSC_PART" value="C440198"/>
 </part>
-<part name="R1" library="rcl" library_urn="urn:adsk.eagle:library:334" deviceset="R-US_" device="R1206" package3d_urn="urn:adsk.eagle:package:23540/2">
-<spice>
-<pinmapping spiceprefix="R">
-<pinmap gate="G$1" pin="1" pinorder="1"/>
-<pinmap gate="G$1" pin="2" pinorder="2"/>
-</pinmapping>
-</spice>
-</part>
-<part name="C3" library="rcl" library_urn="urn:adsk.eagle:library:334" deviceset="C-EU" device="C1210K" package3d_urn="urn:adsk.eagle:package:23683/2"/>
 <part name="HVOUT_TP" library="testpad" library_urn="urn:adsk.eagle:library:385" deviceset="TPSQ" device="PAD1-13" package3d_urn="urn:adsk.eagle:package:27946/1"/>
 <part name="J2" library="Headers" deviceset="61300211121" device="" package3d_urn="urn:adsk.eagle:package:11390690/2"/>
@@
 <wire x1="124.46" y1="91.44" x2="124.46" y2="27.94" width="0.1524" layer="97" style="longdash"/>
 <wire x1="254" y1="91.44" x2="254" y2="27.94" width="0.1524" layer="97" style="longdash"/>
-<text x="55.88" y="38.1" size="1.778" layer="91">snubb</text>
 <text x="127" y="55.88" size="1.778" layer="91">injection</text>
 <polygon width="0.1524" layer="117">
@@
 <instance part="SUPPLY4" gate="GND" x="154.94" y="152.4" smashed="yes"/>
 <instance part="SUPPLY5" gate="GND" x="154.94" y="109.22" smashed="yes"/>
-<instance part="R1" gate="G$1" x="53.34" y="33.02" smashed="yes">
-<attribute name="NAME" x="49.53" y="34.5186" size="1.778" layer="95"/>
-<attribute name="VALUE" x="49.53" y="29.718" size="1.778" layer="96"/>
-</instance>
-<instance part="C3" gate="G$1" x="66.04" y="33.02" smashed="yes" rot="R90">
-<attribute name="NAME" x="65.659" y="34.544" size="1.778" layer="95" rot="R90"/>
-<attribute name="VALUE" x="70.739" y="34.544" size="1.778" layer="96" rot="R90"/>
-</instance>
 <instance part="HVOUT_TP" gate="G$1" x="228.6" y="149.86" smashed="yes" rot="R180">
 <attribute name="NAME" x="233.68" y="154.305" size="1.778" layer="95" rot="R180"/>
@@
 <junction x="50.8" y="60.96"/>
 </segment>
-<segment>
-<pinref part="C3" gate="G$1" pin="2"/>
-<wire x1="71.12" y1="33.02" x2="81.28" y2="33.02" width="0.1524" layer="91"/>
-<label x="73.66" y="33.02" size="1.778" layer="95"/>
-</segment>
 </net>
 <net name="DRAIN1" class="0">
@@
 <wire x1="50.8" y1="68.58" x2="50.8" y2="71.12" width="0.1524" layer="91"/>
 <junction x="50.8" y="71.12"/>
-</segment>
-<segment>
-<pinref part="R1" gate="G$1" pin="1"/>
-<wire x1="48.26" y1="33.02" x2="38.1" y2="33.02" width="0.1524" layer="91"/>
-<label x="35.56" y="33.02" size="1.778" layer="95"/>
 </segment>
 </net>
@@
 <wire x1="83.82" y1="66.04" x2="109.22" y2="66.04" width="0.1524" layer="91"/>
 <label x="99.06" y="66.04" size="1.778" layer="95"/>
-</segment>
-</net>
-<net name="N$29" class="0">
-<segment>
-<pinref part="R1" gate="G$1" pin="2"/>
-<pinref part="C3" gate="G$1" pin="1"/>
-<wire x1="58.42" y1="33.02" x2="63.5" y2="33.02" width="0.1524" layer="91"/>
 </segment>
 </net>
@@
 <attribute name="VALUE" x="186.69" y="69.85" size="1.778" layer="96" align="center-left"/>
 </instance>
-<instance part="GND6" gate="1" x="228.6" y="68.58" smashed="yes"/>
+<instance part="GND6" gate="1" x="243.84" y="63.5" smashed="yes"/>
 <instance part="R3" gate="G$1" x="162.56" y="104.14" smashed="yes">
 <attribute name="NAME" x="158.75" y="105.6386" size="1.778" layer="95"/>
@@
 <attribute name="LCSC_PART" x="86.36" y="149.86" size="1.778" layer="96" display="off"/>
 </instance>
-<instance part="R6" gate="G$1" x="223.52" y="93.98" smashed="yes" rot="R90">
-<attribute name="NAME" x="222.0214" y="90.17" size="1.778" layer="95" rot="R90"/>
-<attribute name="VALUE" x="226.822" y="90.17" size="1.778" layer="96" rot="R90"/>
-</instance>
-<instance part="R5" gate="G$1" x="233.68" y="93.98" smashed="yes" rot="R90">
-<attribute name="NAME" x="232.1814" y="90.17" size="1.778" layer="95" rot="R90"/>
-<attribute name="VALUE" x="236.982" y="90.17" size="1.778" layer="96" rot="R90"/>
+<instance part="R6" gate="G$1" x="238.76" y="88.9" smashed="yes" rot="R90">
+<attribute name="NAME" x="237.2614" y="85.09" size="1.778" layer="95" rot="R90"/>
+<attribute name="VALUE" x="242.062" y="85.09" size="1.778" layer="96" rot="R90"/>
+</instance>
+<instance part="R5" gate="G$1" x="248.92" y="88.9" smashed="yes" rot="R90">
+<attribute name="NAME" x="247.4214" y="85.09" size="1.778" layer="95" rot="R90"/>
+<attribute name="VALUE" x="252.222" y="85.09" size="1.778" layer="96" rot="R90"/>
 </instance>
 <instance part="GND7" gate="1" x="124.46" y="137.16" smashed="yes"/>
@@
 </segment>
 <segment>
-<wire x1="228.6" y1="83.82" x2="228.6" y2="71.12" width="0.1524" layer="91"/>
-<label x="228.6" y="73.66" size="1.778" layer="95" rot="R90"/>
+<wire x1="243.84" y1="78.74" x2="243.84" y2="66.04" width="0.1524" layer="91"/>
+<label x="243.84" y="68.58" size="1.778" layer="95" rot="R90"/>
 <pinref part="GND6" gate="1" pin="GNDA"/>
 <pinref part="R6" gate="G$1" pin="1"/>
-<wire x1="228.6" y1="83.82" x2="223.52" y2="83.82" width="0.1524" layer="91"/>
-<wire x1="223.52" y1="83.82" x2="223.52" y2="88.9" width="0.1524" layer="91"/>
+<wire x1="243.84" y1="78.74" x2="238.76" y2="78.74" width="0.1524" layer="91"/>
+<wire x1="238.76" y1="78.74" x2="238.76" y2="83.82" width="0.1524" layer="91"/>
 <pinref part="R5" gate="G$1" pin="1"/>
-<wire x1="233.68" y1="88.9" x2="233.68" y2="83.82" width="0.1524" layer="91"/>
-<wire x1="233.68" y1="83.82" x2="228.6" y2="83.82" width="0.1524" layer="91"/>
-<junction x="228.6" y="83.82"/>
+<wire x1="248.92" y1="83.82" x2="248.92" y2="78.74" width="0.1524" layer="91"/>
+<wire x1="248.92" y1="78.74" x2="243.84" y2="78.74" width="0.1524" layer="91"/>
+<junction x="243.84" y="78.74"/>
 </segment>
 <segment>
@@
 <net name="BRIDGEGND" class="0">
 <segment>
-<wire x1="228.6" y1="104.14" x2="228.6" y2="119.38" width="0.1524" layer="91"/>
-<wire x1="228.6" y1="119.38" x2="223.52" y2="119.38" width="0.1524" layer="91"/>
-<label x="223.52" y="119.38" size="1.778" layer="95"/>
+<wire x1="243.84" y1="99.06" x2="243.84" y2="114.3" width="0.1524" layer="91"/>
+<wire x1="243.84" y1="114.3" x2="238.76" y2="114.3" width="0.1524" layer="91"/>
+<label x="238.76" y="114.3" size="1.778" layer="95"/>
 <pinref part="R6" gate="G$1" pin="2"/>
-<wire x1="223.52" y1="99.06" x2="223.52" y2="104.14" width="0.1524" layer="91"/>
-<wire x1="223.52" y1="104.14" x2="228.6" y2="104.14" width="0.1524" layer="91"/>
+<wire x1="238.76" y1="93.98" x2="238.76" y2="99.06" width="0.1524" layer="91"/>
+<wire x1="238.76" y1="99.06" x2="243.84" y2="99.06" width="0.1524" layer="91"/>
 <pinref part="R5" gate="G$1" pin="2"/>
-<wire x1="233.68" y1="99.06" x2="233.68" y2="104.14" width="0.1524" layer="91"/>
-<wire x1="233.68" y1="104.14" x2="228.6" y2="104.14" width="0.1524" layer="91"/>
-<junction x="228.6" y="104.14"/>
-</segment>
-<segment>
+<wire x1="248.92" y1="93.98" x2="248.92" y2="99.06" width="0.1524" layer="91"/>
+<wire x1="248.92" y1="99.06" x2="243.84" y2="99.06" width="0.1524" layer="91"/>
+<junction x="243.84" y="99.06"/>
+</segment>
+<segment>
